File: DMH_VCLFO_PCB_1/Breadboard_Layout.kicad_sch (KiCad schematic)
At the start: 0 parts

Commit message: Breadboard troubleshooting changes
Changed lines of the file:
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@@
+		)
+	)
+	(text_box "Tri/Sin"
+		(exclude_from_sim no)
+		(at 66.04 78.74 0)
+		(size 7.62 7.62)
+		(margins 0.9525 0.9525 0.9525 0.9525)
+		(stroke
+			(width 0)
+			(type solid)
+		)
+		(fill
+			(type none)
+		)
+		(effects
+			(font
+				(size 1.27 1.27)
+			)
 		)
 	)
@@
 				(thickness 0.254)
 				(bold yes)
+			)
+		)
+	)
+	(text_box "Rng\nf/ff/s"
+		(exclude_from_sim no)
+		(at 78.74 66.04 0)
+		(size 7.62 7.62)
+		(margins 0.9525 0.9525 0.9525 0.9525)
+		(stroke
+			(width 0)
+			(type solid)
+		)
+		(fill
+			(type none)
+		)
+		(effects
+			(font
+				(size 1.27 1.27)
 			)
 		)
@@
 			)
 		)
+	)
+	(text_box "Pol"
+		(exclude_from_sim no)
+		(at 78.74 78.74 0)
+		(size 7.62 7.62)
+		(margins 0.9525 0.9525 0.9525 0.9525)
+		(stroke
+			(width 0)
+			(type solid)
+		)
+		(fill
+			(type none)
+		)
+		(effects
+			(font
+				(size 1.27 1.27)
+			)
+		)
+	)
+	(text_box "Rnd/Rmp"
+		(exclude_from_sim no)
+		(at 66.04 66.04 0)
+		(size 7.62 7.62)
+		(margins 0.9525 0.9525 0.9525 0.9525)
+		(stroke
+			(width 0)
+			(type solid)
+		)
+		(fill
+			(type none)
+		)
+		(effects
+			(font
+				(size 1.27 1.27)
+			)
+		)
