File: DMH_VCLFO_PCB_1/Core_Circuit.kicad_sch (KiCad schematic)
At the start: 83 parts, among them Q1 BC548, Q2 BC558, Q3 BC548, Q4 BC548, Q5 BS170, Q6 J113, Q7 BC548, U10 TL074, U11 TL074, U12 TL074

Commit message: Breadboard troubleshooting changes
Parts:
- added R84: 100k, Resistor_THT:R_Axial_DIN0207_L6.3mm_D2.5mm_P7.62mm_Horizontal, symbol Device:R_US
- D10, Q3: now fitted
- R37: value 100k -> 51k
Connections:
- net GND: now also R84.2
- net at R37.2, R38.2, U10.12 (+): now also R84.1
Changed lines of the file:
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@@
 	)
 	(junction
+		(at 50.8 24.13)
+		(diameter 0)
+		(color 0 0 0 0)
+	)
+	(junction
 		(at 25.4 101.6)
 		(diameter 0)
@@
 		(stroke
 			(width 0)
-			(type dash)
+			(type default)
 		)
 	)
@@
 		(stroke
 			(width 0)
-			(type dash)
+			(type default)
 		)
 	)
@@
 		(stroke
 			(width 0)
-			(type dash)
+			(type default)
 		)
 	)
@@
 		(stroke
 			(width 0)
-			(type dash)
+			(type default)
 		)
 	)
@@
 	(wire
 		(pts
+			(xy 50.8 17.78) (xy 50.8 24.13)
+		)
+		(stroke
+			(width 0)
+			(type default)
+		)
+	)
+	(wire
+		(pts
 			(xy 250.19 87.63) (xy 250.19 76.2)
 		)
@@
 		(stroke
 			(width 0)
-			(type dash)
+			(type default)
 		)
 	)
@@
 	(wire
 		(pts
+			(xy 76.2 22.86) (xy 76.2 17.78)
+		)
+		(stroke
+			(width 0)
+			(type default)
+		)
+	)
+	(wire
+		(pts
 			(xy 59.69 168.91) (xy 62.23 168.91)
 		)
@@
 		(stroke
 			(width 0)
-			(type dash)
+			(type default)
 		)
 	)
@@
 		(stroke
 			(width 0)
-			(type dash)
+			(type default)
 		)
 	)
@@
 	(wire
 		(pts
+			(xy 76.2 17.78) (xy 67.31 17.78)
+		)
+		(stroke
+			(width 0)
+			(type default)
+		)
+	)
+	(wire
+		(pts
 			(xy 213.36 29.21) (xy 213.36 35.56)
 		)
@@
 	(wire
 		(pts
+			(xy 59.69 17.78) (xy 50.8 17.78)
+		)
+		(stroke
+			(width 0)
+			(type default)
+		)
+	)
+	(wire
+		(pts
 			(xy 187.96 125.73) (xy 181.61 125.73)
 		)
@@
 		(stroke
 			(width 0)
-			(type dash)
+			(type default)
 		)
 	)
@@
 		(in_bom yes)
 		(on_board yes)
-		(dnp yes)
+		(dnp no)
 		(fields_autoplaced yes)
 		(property "Reference" "Q3"
@@
 	)
 	(symbol
+		(lib_id "Device:R_US")
+		(at 63.5 17.78 90)
+		(mirror x)
+		(unit 1)
+		(exclude_from_sim no)
+		(in_bom yes)
+		(on_board no)
+		(dnp no)
+		(property "Reference" "R84"
+			(at 63.754 23.876 90)
+			(effects
+				(font
+					(size 1.27 1.27)
+				)
+			)
+		)
+		(property "Value" "100k"
+			(at 63.754 21.336 90)
+			(effects
+				(font
+					(size 1.27 1.27)
+				)
+			)
+		)
+		(property "Footprint" "Resistor_THT:R_Axial_DIN0207_L6.3mm_D2.5mm_P7.62mm_Horizontal"
+			(at 63.754 18.796 90)
+			(effects
+				(font
+					(size 1.27 1.27)
+				)
+				(hide yes)
+			)
+		)
+		(property "Datasheet" "~"
+			(at 63.5 17.78 0)
+			(effects
+				(font
+					(size 1.27 1.27)
+				)
+				(hide yes)
+			)
+		)
+		(property "Description" "Resistor, US symbol"
+			(at 63.5 17.78 0)
+			(effects
+				(font
+					(size 1.27 1.27)
+				)
+				(hide yes)
+			)
+		)
+		(property "Function" ""
+			(at 63.5 17.78 0)
+			(effects
+				(font
+					(size 1.27 1.27)
+				)
+			)
+		)
+		(pin "1"
+		)
+		(pin "2"
+		)
+		(instances
+			(project "DMH_VCLFO_PCB_1"
+				(path "/58f4306d-5387-4983-bb08-41a2313fd315/7ad2d702-dfb7-4d49-a82d-34430dd5948f"
+					(reference "R84")
+					(unit 1)
+				)
+			)
+		)
+	)
+	(symbol
 		(lib_id "Amplifier_Operational:TL074")
 		(at 140.97 165.1 0)
@@
 		(in_bom yes)
 		(on_board yes)
-		(dnp yes)
+		(dnp no)
 		(fields_autoplaced yes)
 		(property "Reference" "D10"
@@
 	(symbol
 		(lib_id "power:GND")
+		(at 76.2 22.86 0)
+		(unit 1)
+		(exclude_from_sim no)
+		(in_bom yes)
+		(on_board no)
+		(dnp no)
+		(fields_autoplaced yes)
+		(property "Reference" "#PWR070"
+			(at 76.2 29.21 0)
+			(effects
+				(font
+					(size 1.27 1.27)
+				)
+				(hide yes)
+			)
+		)
+		(property "Value" "GND"
+			(at 76.2 27.94 0)
+			(effects
+				(font
+					(size 1.27 1.27)
+				)
+			)
+		)
+		(property "Footprint" ""
+			(at 76.2 22.86 0)
+			(effects
+				(font
+					(size 1.27 1.27)
+				)
+				(hide yes)
+			)
+		)
+		(property "Datasheet" ""
+			(at 76.2 22.86 0)
+			(effects
+				(font
+					(size 1.27 1.27)
+				)
+				(hide yes)
+			)
+		)
+		(property "Description" "Power symbol creates a global label with name \"GND\" , ground"
+			(at 76.2 22.86 0)
+			(effects
+				(font
+					(size 1.27 1.27)
+				)
+				(hide yes)
+			)
+		)
+		(pin "1"
+		)
+		(instances
+			(project "DMH_VCLFO_PCB_1"
+				(path "/58f4306d-5387-4983-bb08-41a2313fd315/7ad2d702-dfb7-4d49-a82d-34430dd5948f"
+					(reference "#PWR070")
+					(unit 1)
+				)
+			)
+		)
+	)
+	(symbol
+		(lib_id "power:GND")
 		(at 109.22 175.26 0)
 		(unit 1)
@@
 			)
 		)
-		(property "Value" "100k"
+		(property "Value" "51k"
 			(at 38.354 27.686 90)
 			(effects

Commit message: Added super fast range option
Parts:
- added C12: 100nF, Capacitor_THT:C_Disc_D4.3mm_W1.9mm_P5.00mm, symbol Device:C
- C7: value 100nF -> 10nF
- R37: value 51k -> 100k
- R84: value 100k -> 680k
Connections:
- net Tri_Raw: now also C12.2
- new net Rng_Sw_3: C12.1
Other:
- moved on the sheet: C7
Changed lines of the file:
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@@
 	)
 	(junction
+		(at 127 43.18)
+		(diameter 0)
+		(color 0 0 0 0)
+	)
+	(junction
 		(at 250.19 76.2)
 		(diameter 0)
@@
 	)
 	(junction
+		(at 127 33.02)
+		(diameter 0)
+		(color 0 0 0 0)
+	)
+	(junction
 		(at 250.19 116.84)
 		(diameter 0)
@@
 	)
 	(junction
+		(at 97.79 43.18)
+		(diameter 0)
+		(color 0 0 0 0)
+	)
+	(junction
 		(at 25.4 166.37)
 		(diameter 0)
@@
 	)
 	(junction
-		(at 127 38.1)
-		(diameter 0)
-		(color 0 0 0 0)
-	)
-	(junction
 		(at 213.36 48.26)
 		(diameter 0)
@@
 	(wire
 		(pts
+			(xy 127 33.02) (xy 127 43.18)
+		)
+		(stroke
+			(width 0)
+			(type default)
+		)
+	)
+	(wire
+		(pts
+			(xy 124.46 33.02) (xy 127 33.02)
+		)
+		(stroke
+			(width 0)
+			(type default)
+		)
+	)
+	(wire
+		(pts
 			(xy 31.75 46.99) (xy 31.75 49.53)
 		)
@@
 	(wire
 		(pts
-			(xy 97.79 25.4) (xy 101.6 25.4)
+			(xy 97.79 27.94) (xy 101.6 27.94)
 		)
 		(stroke
@@
 	(wire
 		(pts
-			(xy 97.79 48.26) (xy 97.79 38.1)
+			(xy 97.79 48.26) (xy 97.79 43.18)
 		)
 		(stroke
@@
 	(wire
 		(pts
-			(xy 127 22.86) (xy 127 38.1)
-		)
-		(stroke
-			(width 0)
-			(type default)
-		)
-	)
-	(wire
-		(pts
 			(xy 139.7 22.86) (xy 127 22.86)
 		)
@@
 	(wire
 		(pts
-			(xy 231.14 44.45) (xy 232.41 44.45)
+			(xy 127 43.18) (xy 127 50.8)
 		)
 		(stroke
@@
 	(wire
 		(pts
-			(xy 21.59 63.5) (xy 25.4 63.5)
+			(xy 231.14 44.45) (xy 232.41 44.45)
 		)
 		(stroke
@@
 	(wire
 		(pts
-			(xy 74.93 114.3) (xy 76.2 114.3)
+			(xy 21.59 63.5) (xy 25.4 63.5)
 		)
 		(stroke
@@
 	(wire
 		(pts
-			(xy 213.36 114.3) (xy 215.9 114.3)
+			(xy 74.93 114.3) (xy 76.2 114.3)
 		)
 		(stroke
@@
 	(wire
 		(pts
-			(xy 232.41 33.02) (xy 250.19 33.02)
+			(xy 213.36 114.3) (xy 215.9 114.3)
 		)
 		(stroke
@@
 	(wire
 		(pts
-			(xy 96.52 129.54) (xy 96.52 130.81)
+			(xy 232.41 33.02) (xy 250.19 33.02)
 		)
 		(stroke
@@
 	(wire
 		(pts
-			(xy 127 38.1) (xy 127 50.8)
+			(xy 96.52 129.54) (xy 96.52 130.81)
 		)
 		(stroke
@@
 	(wire
 		(pts
-			(xy 97.79 38.1) (xy 116.84 38.1)
+			(xy 97.79 43.18) (xy 116.84 43.18)
 		)
 		(stroke
@@
 	(wire
 		(pts
+			(xy 127 22.86) (xy 127 33.02)
+		)
+		(stroke
+			(width 0)
+			(type default)
+		)
+	)
+	(wire
+		(pts
 			(xy 25.4 101.6) (xy 25.4 104.14)
 		)
@@
 	(wire
 		(pts
-			(xy 124.46 38.1) (xy 127 38.1)
+			(xy 124.46 43.18) (xy 127 43.18)
 		)
 		(stroke
@@
 	(wire
 		(pts
-			(xy 97.79 38.1) (xy 97.79 25.4)
+			(xy 97.79 38.1) (xy 97.79 27.94)
 		)
 		(stroke
@@
 	(wire
 		(pts
+			(xy 97.79 43.18) (xy 97.79 38.1)
+		)
+		(stroke
+			(width 0)
+			(type default)
+		)
+	)
+	(wire
+		(pts
 			(xy 25.4 99.06) (xy 25.4 101.6)
 		)
@@
 	(wire
 		(pts
+			(xy 114.3 33.02) (xy 116.84 33.02)
+		)
+		(stroke
+			(width 0)
+			(type default)
+		)
+	)
+	(wire
+		(pts
 			(xy 250.19 76.2) (xy 248.92 76.2)
 		)
@@
 	(hierarchical_label "Rng_Sw_2"
 		(shape output)
-		(at 101.6 25.4 0)
+		(at 101.6 27.94 0)
 		(effects
 			(font
@@
 		)
 	)
+	(hierarchical_label "Rng_Sw_3"
+		(shape input)
+		(at 114.3 33.02 180)
+		(effects
+			(font
+				(size 1.27 1.27)
+			)
+			(justify right)
+		)
+	)
 	(hierarchical_label "Pot In"
 		(shape input)
@@
 	)
 	(symbol
+		(lib_id "Device:C")
+		(at 120.65 33.02 90)
+		(unit 1)
+		(exclude_from_sim no)
+		(in_bom yes)
+		(on_board yes)
+		(dnp no)
+		(property "Reference" "C12"
+			(at 120.65 26.67 90)
+			(effects
+				(font
+					(size 1.27 1.27)
+				)
+			)
+		)
+		(property "Value" "100nF"
+			(at 120.65 29.21 90)
+			(effects
+				(font
+					(size 1.27 1.27)
+				)
+			)
+		)
+		(property "Footprint" "Capacitor_THT:C_Disc_D4.3mm_W1.9mm_P5.00mm"
+			(at 124.46 32.0548 0)
+			(effects
+				(font
+					(size 1.27 1.27)
+				)
+				(hide yes)
+			)
+		)
+		(property "Datasheet" "~"
+			(at 120.65 33.02 0)
+			(effects
+				(font
+					(size 1.27 1.27)
+				)
+				(hide yes)
+			)
+		)
+		(property "Description" "Unpolarized capacitor"
+			(at 120.65 33.02 0)
+			(effects
+				(font
+					(size 1.27 1.27)
+				)
+				(hide yes)
+			)
+		)
+		(pin "1"
+		)
+		(pin "2"
+		)
+		(instances
+			(project "DMH_VCLFO_PCB_1"
+				(path "/58f4306d-5387-4983-bb08-41a2313fd315/7ad2d702-dfb7-4d49-a82d-34430dd5948f"
+					(reference "C12")
+					(unit 1)
+				)
+			)
+		)
+	)
+	(symbol
 		(lib_id "power:GND")
 		(at 171.45 163.83 0)
@@
 			)
 		)
-		(property "Value" "100k"
+		(property "Value" "680k"
 			(at 63.754 21.336 90)
 			(effects
@@
 	(symbol
 		(lib_id "Device:C")
-		(at 120.65 38.1 90)
+		(at 120.65 43.18 90)
 		(unit 1)
 		(exclude_from_sim no)
@@
 		(on_board yes)
 		(dnp no)
-		(fields_autoplaced yes)
 		(property "Reference" "C7"
-			(at 120.65 30.48 90)
+			(at 120.65 36.83 90)
 			(effects
 				(font
@@
 			)
 		)
-		(property "Value" "100nF"
-			(at 120.65 33.02 90)
+		(property "Value" "10nF"
+			(at 120.65 39.37 90)
 			(effects
 				(font
@@
 		)
 		(property "Footprint" "Capacitor_THT:C_Disc_D4.3mm_W1.9mm_P5.00mm"
-			(at 124.46 37.1348 0)
+			(at 124.46 42.2148 0)
 			(effects
 				(font
@@
 		)
 		(property "Datasheet" "~"
-			(at 120.65 38.1 0)
+			(at 120.65 43.18 0)
 			(effects
 				(font
@@
 		)
 		(property "Description" "Unpolarized capacitor"
-			(at 120.65 38.1 0)
+			(at 120.65 43.18 0)
 			(effects
 				(font
@@
 			)
 		)
-		(property "Value" "51k"
+		(property "Value" "100k"
 			(at 38.354 27.686 90)
 			(effects
@@
 		(on_board yes)
 		(dnp no)
-		(fields_autoplaced yes)
 		(property "Reference" "C6"
-			(at 120.65 15.24 90)
+			(at 120.65 16.51 90)
 			(effects
 				(font
@@
 		)
 		(property "Value" "1uF"
-			(at 120.65 17.78 90)
+			(at 120.65 19.05 90)
 			(effects
 				(font
