File: DMH_VCLFO_v2_PCB_Main/Ramp_Shaper_A.kicad_sch (KiCad schematic)
At the start: 10 parts, among them Q7 BC548, U4 TL074

Commit message: Adapted saw shaper
Parts:
- removed C9: 100pF, Capacitor_THT:C_Disc_D4.3mm_W1.9mm_P5.00mm, symbol Device:C
- removed D10: 1N4148, Diode_THT:D_DO-35_SOD27_P7.62mm_Horizontal, symbol Diode:1N4148
- removed Q7: BC548, Package_TO_SOT_THT:TO-92L_Inline_Wide, symbol Transistor_BJT:BC548
- removed R62: 47k, Resistor_THT:R_Axial_DIN0207_L6.3mm_D2.5mm_P7.62mm_Horizontal, symbol Device:R_US
- removed R64, R65, R68: 100k, Resistor_THT:R_Axial_DIN0207_L6.3mm_D2.5mm_P7.62mm_Horizontal, symbol Device:R_US
- removed R74, R77: 10k, Resistor_THT:R_Axial_DIN0207_L6.3mm_D2.5mm_P7.62mm_Horizontal, symbol Device:R_US
- removed U4: TL074, Package_DIP:DIP-14_W7.62mm_Socket, symbol Amplifier_Operational:TL074
