File: DMH_VCLFO_v2_PCB_Main/Random_A.kicad_sch (KiCad schematic)
At the start: 17 parts, among them Q4 BC548, Q6 J113, U3 TL074

Commit message: Replaced sine shaper and adapted random
Parts:
- removed C4: 1uF, Capacitor_THT:C_Disc_D4.3mm_W1.9mm_P5.00mm, symbol Device:C
- removed C5: 1nF, Capacitor_THT:C_Disc_D4.3mm_W1.9mm_P5.00mm, symbol Device:C
- removed C8: 100nF, Capacitor_THT:C_Disc_D4.3mm_W1.9mm_P5.00mm, symbol Device:C
- removed D8, D9: 1N4148, Diode_THT:D_DO-35_SOD27_P7.62mm_Horizontal, symbol Device:D
- removed Q4: BC548, Package_TO_SOT_THT:TO-92_Inline_Wide, symbol Transistor_BJT:BC548
- removed Q6: J113, Package_TO_SOT_THT:TO-92L_Inline, symbol Transistor_FET:MMBFJ113
- removed R47, R50, R55, R58, R60: 100k, Resistor_THT:R_Axial_DIN0207_L6.3mm_D2.5mm_P7.62mm_Horizontal, symbol Device:R_US
- removed R51: 10k, Resistor_THT:R_Axial_DIN0207_L6.3mm_D2.5mm_P7.62mm_Horizontal, symbol Device:R_US
- removed R54: 330R, Resistor_THT:R_Axial_DIN0207_L6.3mm_D2.5mm_P7.62mm_Horizontal, symbol Device:R_US
- removed R57: 33k, Resistor_THT:R_Axial_DIN0207_L6.3mm_D2.5mm_P7.62mm_Horizontal, symbol Device:R_US
- removed R61: 1M, Resistor_THT:R_Axial_DIN0207_L6.3mm_D2.5mm_P7.62mm_Horizontal, symbol Device:R_US
- removed U3: TL074, Package_DIP:DIP-14_W7.62mm_Socket, symbol Amplifier_Operational:TL074
Connections:
- no-connect marks 1 -> 0
