File: DMH_VCLFO_v2_PCB_Main/Breadboard_Layout.kicad_sch (KiCad schematic)
At the start: 0 parts

Commit message: Notes from breadboarding
Changed lines of the file:
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@@
 		)
 	)
-	(text_box "U12\nTL074"
+	(text_box "U11\nTL074"
 		(exclude_from_sim no)
 		(at 114.3 101.6 0)
@@
 		)
 	)
-	(text_box "U11\nTL074"
+	(text_box "U12\nTL074"
 		(exclude_from_sim no)
 		(at 165.1 101.6 0)
