File: DMH_VCLFO_v2_PCB_Main/Core_Circuit.kicad_sch (KiCad schematic)
At the start: 95 parts, among them J11 Conn_02x03_Odd_Even, J110 Conn_02x03_Odd_Even, J12 Conn_02x04_Odd_Even, J120 Conn_02x04_Odd_Even, J13 Conn_02x03_Odd_Even, J130 Conn_02x03_Odd_Even, Q10 BC548, Q11 BC548, Q12 BC558, Q13 BC558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

Commit message: Adjustments on breadboard
Parts:
- C11: value 22nF -> 2x22nF
Other:
- note removed: "22pF in bb"
- note removed: "2k in bb"
Changed lines of the file:
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@@
 		(comment 1 "PCB for 10cm Kosmo format synthesizer module")
 	)
-	(circle
-		(center 294.64 57.15)
-		(radius 6.35)
-		(stroke
-			(width 0)
-			(type default)
-		)
-		(fill
-			(type none)
-		)
-	)
-	(circle
-		(center 340.106 55.626)
-		(radius 6.35)
-		(stroke
-			(width 0)
-			(type default)
-		)
-		(fill
-			(type none)
-		)
-	)
-	(circle
-		(center 172.466 179.324)
-		(radius 6.35)
-		(stroke
-			(width 0)
-			(type default)
-		)
-		(fill
-			(type none)
-		)
-	)
-	(circle
-		(center 133.096 148.844)
-		(radius 6.35)
-		(stroke
-			(width 0)
-			(type default)
-		)
-		(fill
-			(type none)
-		)
-	)
-	(text "22pF in bb"
-		(exclude_from_sim no)
-		(at 133.35 140.97 0)
-		(effects
-			(font
-				(size 1.27 1.27)
-			)
-		)
-	)
-	(text "2k in bb"
-		(exclude_from_sim no)
-		(at 334.264 62.992 0)
-		(effects
-			(font
-				(size 1.27 1.27)
-			)
-		)
-	)
-	(text "22pF in bb"
-		(exclude_from_sim no)
-		(at 172.72 171.45 0)
-		(effects
-			(font
-				(size 1.27 1.27)
-			)
-		)
-	)
-	(text "2k in bb"
-		(exclude_from_sim no)
-		(at 299.974 65.024 0)
-		(effects
-			(font
-				(size 1.27 1.27)
-			)
-		)
-	)
 	(junction
 		(at 339.09 63.5)
@@
 			)
 		)
-		(property "Value" "22nF"
+		(property "Value" "2x22nF"
 			(at 260.35 140.97 90)
 			(effects

Commit message: Rearranged IO page
Parts:
- removed J12, J120: Conn_02x04_Odd_Even, Connector_PinHeader_2.54mm:PinHeader_2x04_P2.54mm_Horizontal, symbol Connector_Generic:Conn_02x04_Odd_Even
- removed R57, R59, R61, R9: 100k, Resistor_THT:R_Axial_DIN0207_L6.3mm_D2.5mm_P7.62mm_Horizontal, symbol Device:R_US
- removed R66: 220k, Resistor_THT:R_Axial_DIN0207_L6.3mm_D2.5mm_P7.62mm_Horizontal, symbol Device:R_US
- added J12: Conn_02x03_Odd_Even, Connector_PinSocket_2.54mm:PinSocket_2x03_P2.54mm_Vertical, symbol Connector_Generic:Conn_02x03_Odd_Even
- added J120: Conn_02x03_Odd_Even, Connector_PinHeader_2.54mm:PinHeader_2x03_P2.54mm_Horizontal, symbol Connector_Generic:Conn_02x03_Odd_Even
- added R5, R6: 1k, Resistor_THT:R_Axial_DIN0207_L6.3mm_D2.5mm_P7.62mm_Horizontal, symbol Device:R_US
- U10: footprint Package_DIP:DIP-14_W7.62mm_Socket -> (none)
Connections:
- net A_VOct_Trim_p12_S is gone; now on an unnamed net: U10.1
- net A_Rng_Sw_p1_M: now also J12.2 (Pin_2)
- net A_Rng_Sw_p1_S: now also J120.2 (Pin_2)
- net A_Rng_Sw_p3_M: now also J12.4 (Pin_4)
- net A_Rng_Sw_p3_S: now also J120.4 (Pin_4)
- net A_Saw_S: now also R5.1; no longer C12.2, R76.2, R77.1, U11.1
- net A_Sqr_S: now also R6.1; no longer R80.1, R81.2
- net A_Sync_M: now also J12.1 (Pin_1)
- net A_Sync_S: now also J120.1 (Pin_1)
- net A_VOct_Trim_p3_M: now also J12.3 (Pin_3)
- net A_VOct_Trim_p3_S: now also J120.3 (Pin_3)
- net GND: now also J12.5 (Pin_5), J12.6 (Pin_6), J120.5 (Pin_5), J120.6 (Pin_6); no longer U10.3 (+)
- net at U10.2 (-): now also R6.2
- new net: C12.2, R5.2, R76.2, R77.1, U11.1
- new net: R80.1, R81.2, U10.3 (+)
