File: DMH_VCLFO_v2_PCB_Main/Inputs_and_Outputs_C.kicad_sch (KiCad schematic)
At the start: 41 parts, among them J1 TS_Jack_6.35mm_Sw, J19 Conn_01x08, J2 TS_Jack_6.35mm_Sw, J20 Conn_01x08, J21 IDA_02x05, J22 Conn_01x08, J23 Conn_01x08, J3 TS_Jack_6.35mm_Sw, J4 TS_Jack_6.35mm_Sw, J5 TS_Jack_6.35mm_Sw, J6 TS_Jack_6.35mm_Sw, Q1 BC548, Q2 BC558, SW1 SW_SPDT, SW2 SPDT_OnOffOn, SW3 SW_SPDT, SW4 SW_SPDT, U1 TL074

Commit message: Prepared for PCB design
Parts:
- J31: renamed from J21; value IDA_02x05 -> IDC_02x05
- RV10: renamed from RV2; footprint SynthStuff:Potentiometer_TT_P110KH1 -> SynthStuff:Potentiometer_Alpha_RD901F-40-00D_Single_Vertical
- RV9: renamed from RV1; footprint SynthStuff:Potentiometer_TT_P110KH1 -> SynthStuff:Potentiometer_Alpha_RD901F-40-00D_Single_Vertical
- U3: renamed from U1; footprint (none) -> Package_DIP:DIP-14_W7.62mm_Socket
- renumbered D1 to D5, D2 to D6, J1 to J13, J2 to J14, J3 to J15, J4 to J16, J5 to J17, J6 to J18, J19 to J29, J20 to J30, J22 to J32, J23 to J33, Q1 to Q5, Q2 to Q6, R1 to R35, R2 to R36, R3 to R37, R4 to R38, R5 to R39, R6 to R40, R7 to R41, R8 to R42, R9 to R43, R10 to R44, R11 to R45, R12 to R46, R13 to R47, R14 to R48, R15 to R49, R16 to R50, R17 to R51, RV3 to RV11, RV4 to RV12, SW2 to SW10, SW3 to SW11, SW4 to SW12, SW1 to SW9, U1 to U3
Connections:
- net A_BusCV_Sw_p2_C renamed C_BusCV_Sw_p2_C
- net A_BusCV_Sw_p2_M renamed C_BusCV_Sw_p2_M
- net A_CV_Amt_Pot_p2_C renamed C_CV_Amt_Pot_p2_C
- net A_CV_Amt_Pot_p2_M renamed C_CV_Amt_Pot_p2_M
- net A_CV_Amt_Pot_p3_C renamed C_CV_Amt_Pot_p3_C
- net A_CV_Amt_Pot_p3_M renamed C_CV_Amt_Pot_p3_M
- net A_FRng_Trim_p2_C renamed C_FRng_Trim_p2_C
- net A_FRng_Trim_p2_M renamed C_FRng_Trim_p2_M
- net A_Freq_Pot_p2_C renamed C_Freq_Pot_p2_C
- net A_Freq_Pot_p2_M renamed C_Freq_Pot_p2_M
- net A_Rmp_C renamed C_Rmp_C
- net A_Rmp_M renamed C_Rmp_M
- net A_Rmp_Rnd_Sw_p2_C renamed C_Rmp_Rnd_Sw_p2_C
- net A_Rmp_Rnd_Sw_p2_M renamed C_Rmp_Rnd_Sw_p2_M
- net A_Rnd_C renamed C_Rnd_C
- net A_Rnd_M renamed C_Rnd_M
- net A_Rng_Sw_p1_C renamed C_Rng_Sw_p1_C
- net A_Rng_Sw_p1_M renamed C_Rng_Sw_p1_M
- net A_Rng_Sw_p3_C renamed C_Rng_Sw_p3_C
- net A_Rng_Sw_p3_M renamed C_Rng_Sw_p3_M
- net A_Saw_M renamed C_Saw_M
- net A_Sin_C renamed C_Sin_C
- net A_Sin_M renamed C_Sin_M
- net A_Sin_Tri_Sw_p2_C renamed C_Sin_Tri_Sw_p2_C
- net A_Sin_Tri_Sw_p2_M renamed C_Sin_Tri_Sw_p2_M
- net A_Sqr_M renamed C_Sqr_M
- net A_Sync_M renamed C_Sync_M
- net A_Tri_C renamed C_Tri_C
- net A_Tri_M renamed C_Tri_M
- net A_VOct_Trim_p12_C renamed C_VOct_Trim_p12_C
- net A_VOct_Trim_p12_M renamed C_VOct_Trim_p12_M
- net A_VOct_Trim_p3_C renamed C_VOct_Trim_p3_C
- net A_VOct_Trim_p3_M renamed C_VOct_Trim_p3_M
