File: DMH_VCLFO_v2_PCB_Main/Sub_module.kicad_sch (KiCad schematic)
At the start: 92 parts, among them J11 Conn_02x03_Odd_Even, J110 Conn_02x03_Odd_Even, J12 Conn_02x03_Odd_Even, J120 Conn_02x03_Odd_Even, J13 Conn_02x03_Odd_Even, J130 Conn_02x03_Odd_Even, Q10 BC548, Q11 BC548, Q12 BC558, Q13 BC558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

Commit message: Prepared for PCB design
Parts:
- renumbered C5 to C1, C14 to C10, C15 to C11, C16 to C12, C17 to C13, C19 to C14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
