File: DMH_VCLFO_v2_PCB_Main/Sub_module_A.kicad_sch (KiCad schematic)
At the start: 92 parts, among them J11 Conn_02x03_Odd_Even, J110 Conn_02x03_Odd_Even, J12 Conn_02x03_Odd_Even, J120 Conn_02x03_Odd_Even, J13 Conn_02x03_Odd_Even, J130 Conn_02x03_Odd_Even, Q10 BC548, Q11 BC548, Q12 BC558, Q13 BC558, Q14 BC548, Q15 MMBFJ113, Q16 MMBFJ113, Q17 BC548, Q18 BC548, Q19 BC548, Q20 J113, U10 TL074, U11 TL074, U12 TL074

Commit message: Prepared for PCB design
Parts:
- Q10: renamed from Q15; footprint Package_TO_SOT_SMD:SOT-23 -> Package_TO_SOT_THT:TO-92L_Inline
- Q17: renamed from Q16; footprint Package_TO_SOT_SMD:SOT-23 -> Package_TO_SOT_THT:TO-92L_Inline
- Q9: renamed from Q20; value J113 -> MMBFJ113
- U10: footprint (none) -> Package_DIP:DIP-14_W7.62mm_Socket
- renumbered C5 to C1, C14 to C10, C15 to C11, C16 to C12, C17 to C13, C19 to C14, C21 to C15, C18 to C16, C20 to C17, C22 to C18, C6 to C2, C7 to C3, C8 to C4, C9 to C5, C10 to C6, C11 to C7, C12 to C8, C13 to C9, J110 to J34, J11 to J35, J120 to J36, J12 to J37, J130 to J38, J13 to J39, Q19 to Q11, Q10 to Q12, Q12 to Q13, Q11 to Q14, Q13 to Q15, Q14 to Q16, Q17 to Q7, Q18 to Q8, R37 to R52, R38 to R53, R39 to R54, R40 to R55, R43 to R56, R44 to R57, R45 to R58, R46 to R59, R47 to R60, R8 to R61, R49 to R62, R50 to R63, R53 to R64, R54 to R65, R55 to R66, R56 to R67, R52 to R68, R58 to R69, R60 to R70, R62 to R71, R13 to R72, R63 to R73, R64 to R74, R65 to R75, R67 to R76, R70 to R77, R71 to R78, R6 to R79, R72 to R80, R76 to R81, R77 to R82, R79 to R83, R80 to R84, R81 to R85, R82 to R86, R83 to R87, R84 to R88, R85 to R89, R86 to R90, R5 to R91, R87 to R92, R88 to R93, R89 to R94, R90 to R95, R91 to R96, RV4 to RV13, RV5 to RV14
