File: DMH_VCLFO_v2_PCB_Main/Sub_module_B.kicad_sch (KiCad schematic)
At the start: 92 parts, among them J11 Conn_02x03_Odd_Even, J110 Conn_02x03_Odd_Even, J12 Conn_02x03_Odd_Even, J120 Conn_02x03_Odd_Even, J13 Conn_02x03_Odd_Even, J130 Conn_02x03_Odd_Even, Q10 BC548, Q11 BC548, Q12 BC558, Q13 BC558, Q14 BC548, Q15 MMBFJ113, Q16 MMBFJ113, Q17 BC548, Q18 BC548, Q19 BC548, Q20 J113, U10 TL074, U11 TL074, U12 TL074

Commit message: Prepared for PCB design
Parts:
- Q20: value J113 -> MMBFJ113
- Q21: renamed from Q15; footprint Package_TO_SOT_SMD:SOT-23 -> Package_TO_SOT_THT:TO-92L_Inline
- Q28: renamed from Q16; footprint Package_TO_SOT_SMD:SOT-23 -> Package_TO_SOT_THT:TO-92L_Inline
- U20: renamed from U10; footprint (none) -> Package_DIP:DIP-14_W7.62mm_Socket
- renumbered C5 to C19, C6 to C20, C7 to C21, C8 to C22, C9 to C23, C10 to C24, C11 to C25, C12 to C26, C13 to C27, C14 to C28, C15 to C29, C16 to C30, C17 to C31, C19 to C32, C21 to C33, C18 to C34, C20 to C35, C22 to C36, D7 to D13, D8 to D14, D9 to D15, D10 to D16, D11 to D17, D12 to D18, J110 to J40, J11 to J41, J120 to J42, J12 to J43, J130 to J44, J13 to J45, Q17 to Q18, Q18 to Q19, Q19 to Q22, Q10 to Q23, Q12 to Q24, Q11 to Q25, Q13 to Q26, Q14 to Q27, R40 to R100, R43 to R101, R44 to R102, R45 to R103, R46 to R104, R47 to R105, R8 to R106, R49 to R107, R50 to R108, R53 to R109, R54 to R110, R55 to R111, R56 to R112, R52 to R113, R58 to R114, R60 to R115, R62 to R116, R13 to R117, R63 to R118, R64 to R119, R65 to R120, R67 to R121, R70 to R122, R71 to R123, R6 to R124, R72 to R125, R76 to R126, R77 to R127, R79 to R128, R80 to R129, R81 to R130, R82 to R131, R83 to R132, R84 to R133, R85 to R134, R86 to R135, R5 to R136, R87 to R137, R88 to R138, R89 to R139, R90 to R140, R91 to R141, R37 to R97, R38 to R98, R39 to R99, RV4 to RV15, RV5 to RV16, TH1 to TH2, U10 to U20, U11 to U21, U12 to U22
Connections:
- net A_Rmp_M renamed B_Rmp_M
- net A_Rmp_S renamed B_Rmp_S
- net A_Rnd_M renamed B_Rnd_M
- net A_Rnd_S renamed B_Rnd_S
- net A_Rng_Sw_p1_M renamed B_Rng_Sw_p1_M
- net A_Rng_Sw_p1_S renamed B_Rng_Sw_p1_S
- net A_Rng_Sw_p3_M renamed B_Rng_Sw_p3_M
- net A_Rng_Sw_p3_S renamed B_Rng_Sw_p3_S
- net A_Saw_M renamed B_Saw_M
- net A_Saw_S renamed B_Saw_S
- net A_Sin_M renamed B_Sin_M
- net A_Sin_S renamed B_Sin_S
- net A_Sqr_M renamed B_Sqr_M
- net A_Sqr_S renamed B_Sqr_S
- net A_Sync_M renamed B_Sync_M
- net A_Sync_S renamed B_Sync_S
- net A_Tri_M renamed B_Tri_M
- net A_Tri_S renamed B_Tri_S
- net A_VOct_Trim_p3_M renamed B_VOct_Trim_p3_M
- net A_VOct_Trim_p3_S renamed B_VOct_Trim_p3_S
