File: DMH_VCLFO_v2_PCB_Main/Sub_module_C.kicad_sch (KiCad schematic)
At the start: 92 parts, among them J11 Conn_02x03_Odd_Even, J110 Conn_02x03_Odd_Even, J12 Conn_02x03_Odd_Even, J120 Conn_02x03_Odd_Even, J13 Conn_02x03_Odd_Even, J130 Conn_02x03_Odd_Even, Q10 BC548, Q11 BC548, Q12 BC558, Q13 BC558, Q14 BC548, Q15 MMBFJ113, Q16 MMBFJ113, Q17 BC548, Q18 BC548, Q19 BC548, Q20 J113, U10 TL074, U11 TL074, U12 TL074

Commit message: Prepared for PCB design
Parts:
- Q31: renamed from Q20; value J113 -> MMBFJ113
- Q32: renamed from Q15; footprint Package_TO_SOT_SMD:SOT-23 -> Package_TO_SOT_THT:TO-92L_Inline
- Q39: renamed from Q16; footprint Package_TO_SOT_SMD:SOT-23 -> Package_TO_SOT_THT:TO-92L_Inline
- U30: renamed from U10; footprint (none) -> Package_DIP:DIP-14_W7.62mm_Socket
- renumbered C5 to C37, C6 to C38, C7 to C39, C8 to C40, C9 to C41, C10 to C42, C11 to C43, C12 to C44, C13 to C45, C14 to C46, C15 to C47, C16 to C48, C17 to C49, C19 to C50, C21 to C51, C18 to C52, C20 to C53, C22 to C54, D7 to D19, D8 to D20, D9 to D21, D10 to D22, D11 to D23, D12 to D24, J110 to J46, J11 to J47, J120 to J48, J12 to J49, J130 to J50, J13 to J51, Q17 to Q29, Q18 to Q30, Q19 to Q33, Q10 to Q34, Q12 to Q35, Q11 to Q36, Q13 to Q37, Q14 to Q38, R37 to R142, R38 to R143, R39 to R144, R40 to R145, R43 to R146, R44 to R147, R45 to R148, R46 to R149, R47 to R150, R8 to R151, R49 to R152, R50 to R153, R53 to R154, R54 to R155, R55 to R156, R56 to R157, R52 to R158, R58 to R159, R60 to R160, R62 to R161, R13 to R162, R63 to R163, R64 to R164, R65 to R165, R67 to R166, R70 to R167, R71 to R168, R6 to R169, R72 to R170, R76 to R171, R77 to R172, R79 to R173, R80 to R174, R81 to R175, R82 to R176, R83 to R177, R84 to R178, R85 to R179, R86 to R180, R5 to R181, R87 to R182, R88 to R183, R89 to R184, R90 to R185, R91 to R186, RV4 to RV17, RV5 to RV18, TH1 to TH3, U10 to U30, U11 to U31, U12 to U32
Connections:
- net A_Rmp_M renamed C_Rmp_M
- net A_Rmp_S renamed C_Rmp_S
- net A_Rnd_M renamed C_Rnd_M
- net A_Rnd_S renamed C_Rnd_S
- net A_Rng_Sw_p1_M renamed C_Rng_Sw_p1_M
- net A_Rng_Sw_p1_S renamed C_Rng_Sw_p1_S
- net A_Rng_Sw_p3_M renamed C_Rng_Sw_p3_M
- net A_Rng_Sw_p3_S renamed C_Rng_Sw_p3_S
- net A_Saw_M renamed C_Saw_M
- net A_Saw_S renamed C_Saw_S
- net A_Sin_M renamed C_Sin_M
- net A_Sin_S renamed C_Sin_S
- net A_Sqr_M renamed C_Sqr_M
- net A_Sqr_S renamed C_Sqr_S
- net A_Sync_M renamed C_Sync_M
- net A_Sync_S renamed C_Sync_S
- net A_Tri_M renamed C_Tri_M
- net A_Tri_S renamed C_Tri_S
- net A_VOct_Trim_p3_M renamed C_VOct_Trim_p3_M
- net A_VOct_Trim_p3_S renamed C_VOct_Trim_p3_S
