File: DMH_VCLFO_v2_PCB_Main/Inputs_and_Outputs_B.kicad_sch (KiCad schematic)
At the start: 41 parts, among them J1 TS_Jack_6.35mm_Sw, J19 Conn_01x08, J2 TS_Jack_6.35mm_Sw, J20 Conn_01x08, J21 IDA_02x05, J22 Conn_01x08, J23 Conn_01x08, J3 TS_Jack_6.35mm_Sw, J4 TS_Jack_6.35mm_Sw, J5 TS_Jack_6.35mm_Sw, J6 TS_Jack_6.35mm_Sw, Q1 BC548, Q2 BC558, SW1 SW_SPDT, SW2 SPDT_OnOffOn, SW3 SW_SPDT, SW4 SW_SPDT, U1 TL074

Commit message: Prepared for PCB design
Parts:
- J26: renamed from J21; value IDA_02x05 -> IDC_02x05
- RV5: renamed from RV1; footprint SynthStuff:Potentiometer_TT_P110KH1 -> SynthStuff:Potentiometer_Alpha_RD901F-40-00D_Single_Vertical
- RV6: renamed from RV2; footprint SynthStuff:Potentiometer_TT_P110KH1 -> SynthStuff:Potentiometer_Alpha_RD901F-40-00D_Single_Vertical
- U2: renamed from U1; footprint (none) -> Package_DIP:DIP-14_W7.62mm_Socket
- renumbered D1 to D3, D2 to D4, J4 to J10, J5 to J11, J6 to J12, J19 to J24, J20 to J25, J22 to J27, J23 to J28, J1 to J7, J2 to J8, J3 to J9, Q1 to Q3, Q2 to Q4, R1 to R18, R2 to R19, R3 to R20, R4 to R21, R5 to R22, R6 to R23, R7 to R24, R8 to R25, R9 to R26, R10 to R27, R11 to R28, R12 to R29, R13 to R30, R14 to R31, R15 to R32, R16 to R33, R17 to R34, RV3 to RV7, RV4 to RV8, SW1 to SW5, SW2 to SW6, SW3 to SW7, SW4 to SW8, U1 to U2
Connections:
- net A_BusCV_Sw_p2_C renamed B_BusCV_Sw_p2_C
- net A_BusCV_Sw_p2_M renamed B_BusCV_Sw_p2_M
- net A_CV_Amt_Pot_p2_C renamed B_CV_Amt_Pot_p2_C
- net A_CV_Amt_Pot_p2_M renamed B_CV_Amt_Pot_p2_M
- net A_CV_Amt_Pot_p3_C renamed B_CV_Amt_Pot_p3_C
- net A_CV_Amt_Pot_p3_M renamed B_CV_Amt_Pot_p3_M
- net A_FRng_Trim_p2_C renamed B_FRng_Trim_p2_C
- net A_FRng_Trim_p2_M renamed B_FRng_Trim_p2_M
- net A_Freq_Pot_p2_C renamed B_Freq_Pot_p2_C
- net A_Freq_Pot_p2_M renamed B_Freq_Pot_p2_M
- net A_Rmp_C renamed B_Rmp_C
- net A_Rmp_M renamed B_Rmp_M
- net A_Rmp_Rnd_Sw_p2_C renamed B_Rmp_Rnd_Sw_p2_C
- net A_Rmp_Rnd_Sw_p2_M renamed B_Rmp_Rnd_Sw_p2_M
- net A_Rnd_C renamed B_Rnd_C
- net A_Rnd_M renamed B_Rnd_M
- net A_Rng_Sw_p1_C renamed B_Rng_Sw_p1_C
- net A_Rng_Sw_p1_M renamed B_Rng_Sw_p1_M
- net A_Rng_Sw_p3_C renamed B_Rng_Sw_p3_C
- net A_Rng_Sw_p3_M renamed B_Rng_Sw_p3_M
- net A_Saw_M renamed B_Saw_M
- net A_Sin_C renamed B_Sin_C
- net A_Sin_M renamed B_Sin_M
- net A_Sin_Tri_Sw_p2_C renamed B_Sin_Tri_Sw_p2_C
- net A_Sin_Tri_Sw_p2_M renamed B_Sin_Tri_Sw_p2_M
- net A_Sqr_M renamed B_Sqr_M
- net A_Sync_M renamed B_Sync_M
- net A_Tri_C renamed B_Tri_C
- net A_Tri_M renamed B_Tri_M
- net A_VOct_Trim_p12_C renamed B_VOct_Trim_p12_C
- net A_VOct_Trim_p12_M renamed B_VOct_Trim_p12_M
- net A_VOct_Trim_p3_C renamed B_VOct_Trim_p3_C
- net A_VOct_Trim_p3_M renamed B_VOct_Trim_p3_M

Commit message: Main PCB comp placement in progress
Parts:
- J10: Function Out A Saw -> Out B Saw
- J11: Function Out A Rmp/Rnd -> Out B Rmp/Rnd
- J12: Function Out A Sin/Tri -> Out B Sin/Tri
- J24, J25: footprint Connector_PinHeader_2.54mm:PinHeader_1x08_P2.54mm_Vertical -> Connector_PinSocket_2.54mm:PinSocket_1x08_P2.54mm_Vertical
- J7: Function CV In A -> CV In B
- J8: Function Sync A -> Sync B
- J9: Function Out A Sqr -> Out B Sqr
- RV5: Function CV A Amt -> CV B Amt
- RV6: Function Freq A -> Freq B
Connections:
- net B_BusCV_Sw_p2_C: now also J25.4 (Pin_4); no longer J25.7 (Pin_7)
- net B_BusCV_Sw_p2_M: now also J28.4 (Pin_4); no longer J28.7 (Pin_7)
- net B_CV_Amt_Pot_p2_C: now also J24.6 (Pin_6); no longer J24.4 (Pin_4)
- net B_CV_Amt_Pot_p2_M: now also J27.6 (Pin_6); no longer J27.4 (Pin_4)
- net B_FRng_Trim_p2_C: now also J24.1 (Pin_1); no longer J24.6 (Pin_6)
- net B_FRng_Trim_p2_M: now also J27.1 (Pin_1); no longer J27.6 (Pin_6)
- net B_Freq_Pot_p2_C: now also J24.4 (Pin_4); no longer J24.3 (Pin_3)
- net B_Freq_Pot_p2_M: now also J27.4 (Pin_4); no longer J27.3 (Pin_3)
- net B_Rmp_C: now also SW7.3 (C); no longer SW7.1 (A)
- net B_Rnd_C: now also SW7.1 (A); no longer SW7.3 (C)
- net B_Rng_Sw_p1_C: now also J24.3 (Pin_3); no longer J24.1 (Pin_1)
- net B_Rng_Sw_p1_M: now also J27.3 (Pin_3); no longer J27.1 (Pin_1)
- net B_Sin_C: now also J25.6 (Pin_6), SW8.3 (C); no longer J25.4 (Pin_4), SW8.1 (A)
- net B_Sin_M: now also J28.6 (Pin_6); no longer J28.4 (Pin_4)
- net B_Sin_Tri_Sw_p2_C: now also J25.7 (Pin_7); no longer J25.5 (Pin_5)
- net B_Sin_Tri_Sw_p2_M: now also J28.7 (Pin_7); no longer J28.5 (Pin_5)
- net B_Tri_C: now also J25.8 (Pin_8), SW8.1 (A); no longer J25.6 (Pin_6), SW8.3 (C)
- net B_Tri_M: now also J28.8 (Pin_8); no longer J28.6 (Pin_6)
- net B_VOct_Trim_p12_C: now also J24.8 (Pin_8); no longer J24.7 (Pin_7)
- net B_VOct_Trim_p12_M: now also J27.8 (Pin_8); no longer J27.7 (Pin_7)
- net B_VOct_Trim_p3_C: now also J24.7 (Pin_7); no longer J24.8 (Pin_8)
- net B_VOct_Trim_p3_M: now also J27.7 (Pin_7); no longer J27.8 (Pin_8)
- net Bus_CV_C: now also J25.5 (Pin_5), SW5.1 (A); no longer J25.8 (Pin_8), SW5.3 (C)
- net Bus_CV_M: now also J28.5 (Pin_5); no longer J28.8 (Pin_8)
- net Out A Rmp/Rnd TN renamed Out B Rmp/Rnd TN
- net Out A Saw TN renamed Out B Saw TN
- net Out A Sin/Tri TN renamed Out B Sin/Tri TN
- net Out A Sqr TN renamed Out B Sqr TN
- net Sync A TN renamed Sync B TN

Commit message: Main PCB placement done
Parts:
- removed J26: IDC_02x05, SynthStuff:IDC-Header_2x05_P2.54mm_Vertical_BackBone, symbol SynthStuff:BackBone_Connector_10Pin
Connections:
- net Out B Rmp/Rnd TN: no longer names the net of J11.TN
- net Out B Saw TN: no longer names the net of J10.TN
- net Out B Sin/Tri TN renamed B_Out_Sin_Tri_TN_M
- net Out B Sqr TN renamed B_Out_Sqr_TN_M
- net Sync B TN renamed B_Sync_TN_M
- no-connect marks 2 -> 3

Commit message: Main PCB routing done
Parts:
- J11: Function Out B Rmp/Rnd -> Out B R/R
- J12: Function Out B Sin/Tri -> Out B S/T
Changed lines of the file:
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@@
 			)
 		)
-		(property "Function" "Out B Sin/Tri"
+		(property "Function" "Out B S/T"
 			(at 228.6 119.888 0)
 			(effects
@@
 			)
 		)
-		(property "Function" "Out B Rmp/Rnd"
+		(property "Function" "Out B R/R"
 			(at 228.6 145.288 0)
 			(effects

Commit message: Added project with Single VCLFO schematic
Other:
- note removed: "U10A in BB"
- note removed: "U12B in BB"
- note removed: "U12D in BB"
Changed lines of the file:
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@@
 		(comment 1 "PCB for 10cm Kosmo format synthesizer module")
-	)
-	(circle
-		(center 236.22 66.294)
-		(radius 3.81)
-		(stroke
-			(width 0)
-			(type default)
-		)
-		(fill
-			(type none)
-		)
-	)
-	(circle
-		(center 167.64 48.514)
-		(radius 3.81)
-		(stroke
-			(width 0)
-			(type default)
-		)
-		(fill
-			(type none)
-		)
-	)
-	(circle
-		(center 167.64 23.114)
-		(radius 3.81)
-		(stroke
-			(width 0)
-			(type default)
-		)
-		(fill
-			(type none)
-		)
-	)
-	(text "U12B in BB"
-		(exclude_from_sim no)
-		(at 167.64 43.18 0)
-		(effects
-			(font
-				(size 1.27 1.27)
-			)
-		)
-	)
-	(text "U10A in BB"
-		(exclude_from_sim no)
-		(at 243.84 62.23 0)
-		(effects
-			(font
-				(size 1.27 1.27)
-			)
-		)
-	)
-	(text "U12D in BB"
-		(exclude_from_sim no)
-		(at 167.64 17.78 0)
-		(effects
-			(font
-				(size 1.27 1.27)
-			)
-		)
 	)
 	(junction
