File: DMH_VCLFO_v2_PCB_Controls/Core_Circuit.kicad_sch (KiCad schematic)
At the start: 93 parts, among them J46 Conn_02x03_Odd_Even, J47 Conn_02x03_Odd_Even, J48 Conn_02x03_Odd_Even, J49 Conn_02x03_Odd_Even, J50 Conn_02x03_Odd_Even, J51 Conn_02x03_Odd_Even, Q29 BC548, Q30 BC548, Q31 MMBFJ113, Q32 MMBFJ113, Q33 BC548, Q34 BC548, Q35 BC558, Q36 BC548, Q37 BC558, Q38 BC548, Q39 MMBFJ113, U30 TL074, U31 TL074, U32 TL074

Commit message: Controls PCB comp placement in progress
Parts:
- removed C65: 22nF, Capacitor_THT:C_Disc_D4.3mm_W1.9mm_P5.00mm, symbol Device:C
- C11: renamed from C43; value 22nF -> 2x22nF
- Q15: renamed from Q32; footprint Package_TO_SOT_THT:TO-92L_Inline -> Package_TO_SOT_SMD:SOT-23
- Q16: renamed from Q39; footprint Package_TO_SOT_THT:TO-92L_Inline -> Package_TO_SOT_SMD:SOT-23
- Q20: renamed from Q31; value MMBFJ113 -> J113
- U10: renamed from U30; footprint Package_DIP:DIP-14_W7.62mm_Socket -> (none)
- renumbered C42 to C10, C44 to C12, C45 to C13, C46 to C14, C47 to C15, C48 to C16, C49 to C17, C52 to C18, C50 to C19, C53 to C20, C51 to C21, C54 to C22, C37 to C5, C38 to C6, C39 to C7, C40 to C8, C41 to C9, D22 to D10, D23 to D11, D24 to D12, D19 to D7, D20 to D8, D21 to D9, J47 to J11, J46 to J110, J49 to J12, J48 to J120, J51 to J13, J50 to J130, Q34 to Q10, Q36 to Q11, Q35 to Q12, Q37 to Q13, Q38 to Q14, Q29 to Q17, Q30 to Q18, Q33 to Q19, R162 to R13, R142 to R37, R143 to R38, R144 to R39, R145 to R40, R146 to R43, R147 to R44, R148 to R45, R149 to R46, R150 to R47, R152 to R49, R181 to R5, R153 to R50, R158 to R52, R154 to R53, R155 to R54, R156 to R55, R157 to R56, R159 to R58, R169 to R6, R160 to R60, R161 to R62, R163 to R63, R164 to R64, R165 to R65, R166 to R67, R167 to R70, R168 to R71, R170 to R72, R171 to R76, R172 to R77, R173 to R79, R151 to R8, R174 to R80, R175 to R81, R176 to R82, R177 to R83, R178 to R84, R179 to R85, R180 to R86, R182 to R87, R183 to R88, R184 to R89, R185 to R90, R186 to R91, RV17 to RV4, RV18 to RV5, TH3 to TH1, U30 to U10, U31 to U11, U32 to U12
Connections:
- net C_Rmp_M renamed A_Rmp_M
- net C_Rmp_S renamed A_Rmp_S
- net C_Rnd_M renamed A_Rnd_M
- net C_Rnd_S renamed A_Rnd_S
- net C_Rng_Sw_p1_M renamed A_Rng_Sw_p1_M
- net C_Rng_Sw_p1_S renamed A_Rng_Sw_p1_S
- net C_Rng_Sw_p3_M renamed A_Rng_Sw_p3_M
- net C_Rng_Sw_p3_S renamed A_Rng_Sw_p3_S
- net C_Saw_M renamed A_Saw_M
- net C_Saw_S renamed A_Saw_S
- net C_Sin_M renamed A_Sin_M
- net C_Sin_S renamed A_Sin_S
- net C_Sqr_M renamed A_Sqr_M
- net C_Sqr_S renamed A_Sqr_S
- net C_Sync_M renamed A_Sync_M
- net C_Sync_S renamed A_Sync_S
- net C_Tri_M renamed A_Tri_M
- net C_Tri_S renamed A_Tri_S
- net C_VOct_Trim_p3_M renamed A_VOct_Trim_p3_M
- net C_VOct_Trim_p3_S renamed A_VOct_Trim_p3_S
Other:
- moved on the sheet: C11, C9, Q15
