File: DMH_VCLFO_v2_PCB_Controls/Sub_module.kicad_sch (KiCad schematic)
At the start: 93 parts, among them J46 Conn_02x03_Odd_Even, J47 Conn_02x03_Odd_Even, J48 Conn_02x03_Odd_Even, J49 Conn_02x03_Odd_Even, J50 Conn_02x03_Odd_Even, J51 Conn_02x03_Odd_Even, Q29 BC548, Q30 BC548, Q31 MMBFJ113, Q32 MMBFJ113, Q33 BC548, Q34 BC548, Q35 BC558, Q36 BC548, Q37 BC558, Q38 BC548, Q39 MMBFJ113, U30 TL074, U31 TL074, U32 TL074

Commit message: Controls PCB comp placement in progress
Parts:
- removed C65: 22nF, Capacitor_THT:C_Disc_D4.3mm_W1.9mm_P5.00mm, symbol Device:C
- C7: renamed from C43; value 22nF -> 2x22nF
- Q10: renamed from Q32; footprint Package_TO_SOT_THT:TO-92L_Inline -> Package_TO_SOT_SMD:SOT-23
- Q17: renamed from Q39; footprint Package_TO_SOT_THT:TO-92L_Inline -> Package_TO_SOT_SMD:SOT-23
- Q9: renamed from Q31; value MMBFJ113 -> J113
- U10: renamed from U30; footprint Package_DIP:DIP-14_W7.62mm_Socket -> (none)
- renumbered C37 to C1, C46 to C10, C47 to C11, C48 to C12, C49 to C13, C50 to C14, C51 to C15, C52 to C16, C53 to C17, C54 to C18, C38 to C2, C39 to C3, C40 to C4, C41 to C5, C42 to C6, C44 to C8, C45 to C9, D22 to D10, D23 to D11, D24 to D12, D19 to D7, D20 to D8, D21 to D9, J46 to J34, J47 to J35, J48 to J36, J49 to J37, J50 to J38, J51 to J39, Q33 to Q11, Q34 to Q12, Q35 to Q13, Q36 to Q14, Q37 to Q15, Q38 to Q16, Q29 to Q7, Q30 to Q8, R142 to R52, R143 to R53, R144 to R54, R145 to R55, R146 to R56, R147 to R57, R148 to R58, R149 to R59, R150 to R60, R151 to R61, R152 to R62, R153 to R63, R154 to R64, R155 to R65, R156 to R66, R157 to R67, R158 to R68, R159 to R69, R160 to R70, R161 to R71, R162 to R72, R163 to R73, R164 to R74, R165 to R75, R166 to R76, R167 to R77, R168 to R78, R169 to R79, R170 to R80, R171 to R81, R172 to R82, R173 to R83, R174 to R84, R175 to R85, R176 to R86, R177 to R87, R178 to R88, R179 to R89, R180 to R90, R181 to R91, R182 to R92, R183 to R93, R184 to R94, R185 to R95, R186 to R96, RV17 to RV13, RV18 to RV14, TH3 to TH1, U30 to U10, U31 to U11, U32 to U12
Connections:
- net C_Rmp_M renamed A_Rmp_M
- net C_Rmp_S renamed A_Rmp_S
- net C_Rnd_M renamed A_Rnd_M
- net C_Rnd_S renamed A_Rnd_S
- net C_Rng_Sw_p1_M renamed A_Rng_Sw_p1_M
- net C_Rng_Sw_p1_S renamed A_Rng_Sw_p1_S
- net C_Rng_Sw_p3_M renamed A_Rng_Sw_p3_M
- net C_Rng_Sw_p3_S renamed A_Rng_Sw_p3_S
- net C_Saw_M renamed A_Saw_M
- net C_Saw_S renamed A_Saw_S
- net C_Sin_M renamed A_Sin_M
- net C_Sin_S renamed A_Sin_S
- net C_Sqr_M renamed A_Sqr_M
- net C_Sqr_S renamed A_Sqr_S
- net C_Sync_M renamed A_Sync_M
- net C_Sync_S renamed A_Sync_S
- net C_Tri_M renamed A_Tri_M
- net C_Tri_S renamed A_Tri_S
- net C_VOct_Trim_p3_M renamed A_VOct_Trim_p3_M
- net C_VOct_Trim_p3_S renamed A_VOct_Trim_p3_S
Other:
- moved on the sheet: C5, C7, Q10
