File: DMH_VCLFO_v2_PCB_Submodule/Sub_module_A.kicad_sch (KiCad schematic)
At the start: 93 parts, among them J34 Conn_02x03_Odd_Even, J35 Conn_02x03_Odd_Even, J36 Conn_02x03_Odd_Even, J37 Conn_02x03_Odd_Even, J38 Conn_02x03_Odd_Even, J39 Conn_02x03_Odd_Even, Q10 MMBFJ113, Q11 BC548, Q12 BC548, Q13 BC558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

Commit message: Submodule comp placement started
Parts:
- C2, C8, C9: footprint Capacitor_THT:C_Disc_D4.3mm_W1.9mm_P5.00mm -> Capacitor_THT:C_Disc_D3.0mm_W2.0mm_P2.50mm
- Q10, Q17, Q9: value MMBFJ113 -> J113
Changed lines of the file:
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@@
 		(exclude_from_sim no)
 		(in_bom yes)
-		(on_board no)
+		(on_board yes)
 		(dnp no)
 		(fields_autoplaced yes)
@@
 			)
 		)
-		(property "Footprint" "Capacitor_THT:C_Disc_D4.3mm_W1.9mm_P5.00mm"
+		(property "Footprint" "Capacitor_THT:C_Disc_D3.0mm_W2.0mm_P2.50mm"
 			(at 54.3052 66.04 0)
 			(effects
@@
 			)
 		)
-		(property "Value" "MMBFJ113"
+		(property "Value" "J113"
 			(at 113.03 196.85 90)
 			(effects
@@
 			)
 		)
-		(property "Value" "MMBFJ113"
+		(property "Value" "J113"
 			(at 260.35 104.14 90)
 			(effects
@@
 		(exclude_from_sim no)
 		(in_bom yes)
-		(on_board no)
+		(on_board yes)
 		(dnp no)
 		(fields_autoplaced yes)
@@
 		(exclude_from_sim no)
 		(in_bom yes)
-		(on_board no)
+		(on_board yes)
 		(dnp no)
 		(fields_autoplaced yes)
@@
 			)
 		)
-		(property "Footprint" "Capacitor_THT:C_Disc_D4.3mm_W1.9mm_P5.00mm"
+		(property "Footprint" "Capacitor_THT:C_Disc_D3.0mm_W2.0mm_P2.50mm"
 			(at 264.16 149.5552 0)
 			(effects
@@
 			)
 		)
-		(property "Footprint" "Capacitor_THT:C_Disc_D4.3mm_W1.9mm_P5.00mm"
+		(property "Footprint" "Capacitor_THT:C_Disc_D3.0mm_W2.0mm_P2.50mm"
 			(at 340.36 143.8148 0)
 			(effects
@@
 			)
 		)
-		(property "Value" "MMBFJ113"
+		(property "Value" "J113"
 			(at 88.9 100.33 90)
 			(effects

Commit message: Submodule com placement done
Parts:
- TH1: value 10k 3380K -> 10k3380
Connections:
- net A_Rnd_S: now also U12.8, U12.9 (-); no longer U12.6 (-), U12.7
- net Comp_Ref: now also U12.2 (-); no longer U12.13 (-)
- net at D10.1 (K): now also U12.1; no longer U12.14
- net at Q9.1 (D), R71.1, R75.1: now also U12.14; no longer U12.1
- net at R71.2, R74.1: now also U12.13 (-); no longer U12.2 (-)
- net at R54.2, R61.1: now also U12.7; no longer U12.8
- net at C3.2, R73.1: now also U12.12 (+); no longer U12.3 (+)
- net at Q7.1 (C), R54.1, R56.2: now also U12.6 (-); no longer U12.9 (-)
- net at Q8.1 (C), R57.2, R66.1: now also U12.5 (+); no longer U12.10 (+)
- net at C6.1, R78.1: now also U12.3 (+); no longer U12.12 (+)
- net at C4.1, Q9.2 (S): now also U12.10 (+); no longer U12.5 (+)
Changed lines of the file:
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@@
 			)
 		)
+		(property "Function" ""
+			(at 243.84 254 0)
+			(effects
+				(font
+					(size 1.27 1.27)
+				)
+			)
+		)
 		(pin "10"
 		)
@@
 		(exclude_from_sim no)
 		(in_bom yes)
-		(on_board yes)
+		(on_board no)
 		(dnp no)
 		(fields_autoplaced yes)
@@
 		(lib_id "Amplifier_Operational:TL074")
 		(at 69.85 95.25 0)
-		(unit 1)
+		(unit 4)
 		(exclude_from_sim no)
 		(in_bom yes)
@@
 				(path "/58f4306d-5387-4983-bb08-41a2313fd315/7ad2d702-dfb7-4d49-a82d-34430dd5948f"
 					(reference "U12")
-					(unit 1)
+					(unit 4)
 				)
 			)
@@
 		(exclude_from_sim no)
 		(in_bom yes)
-		(on_board yes)
+		(on_board no)
 		(dnp no)
 		(fields_autoplaced yes)
@@
 		(exclude_from_sim no)
 		(in_bom yes)
-		(on_board yes)
+		(on_board no)
 		(dnp no)
 		(fields_autoplaced yes)
@@
 		(lib_id "Amplifier_Operational:TL074")
 		(at 69.85 129.54 0)
-		(unit 4)
+		(unit 1)
 		(exclude_from_sim no)
 		(in_bom yes)
@@
 				(path "/58f4306d-5387-4983-bb08-41a2313fd315/7ad2d702-dfb7-4d49-a82d-34430dd5948f"
 					(reference "U12")
-					(unit 4)
+					(unit 1)
 				)
 			)
@@
 		(at 360.68 40.64 0)
 		(mirror x)
-		(unit 3)
+		(unit 2)
 		(exclude_from_sim no)
 		(in_bom yes)
@@
 				(path "/58f4306d-5387-4983-bb08-41a2313fd315/7ad2d702-dfb7-4d49-a82d-34430dd5948f"
 					(reference "U12")
-					(unit 3)
+					(unit 2)
 				)
 			)
@@
 			)
 		)
-		(property "Value" "10k 3380K"
+		(property "Value" "10k3380"
 			(at 212.09 122.2374 0)
 			(effects
@@
 		(lib_id "Amplifier_Operational:TL074")
 		(at 114.3 116.84 0)
-		(unit 2)
+		(unit 3)
 		(exclude_from_sim no)
 		(in_bom yes)
@@
 				(path "/58f4306d-5387-4983-bb08-41a2313fd315/7ad2d702-dfb7-4d49-a82d-34430dd5948f"
 					(reference "U12")
-					(unit 2)
+					(unit 3)
 				)
 			)
